File: PCB/Design1.sch (EAGLE design)
At the start: 39 parts, among them J1 FTDI_DEVICE, U1 ATMEGA2560AU, Y1 16MHZ

Commit message: Move componets to (hopefully) final location
Connections:
- removed net VCC: D1.C, R2.2
- net 5V: now also D1.C, R2.2
Changed lines of the file:
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@@
 <part name="J1" library="SparkFun-Connectors" deviceset="FTDI_DEVICE" device=""/>
 <part name="D1" library="SparkFun-DiscreteSemi" deviceset="DIODE" device="SMA-ALT"/>
-<part name="SUPPLY4" library="SparkFun-Aesthetics" deviceset="VCC" device=""/>
 <part name="GND4" library="SparkFun-Aesthetics" deviceset="GND" device=""/>
 <part name="LOGO1" library="SparkFun-Aesthetics" deviceset="OSHW-LOGO" device="M" value="OSHW-LOGOM"/>
@@
 <part name="GND8" library="SparkFun-Aesthetics" deviceset="GND" device=""/>
 <part name="SUPPLY7" library="SparkFun-Aesthetics" deviceset="5V" device=""/>
+<part name="SUPPLY4" library="SparkFun-Aesthetics" deviceset="5V" device=""/>
 </parts>
 <sheets>
@@
 <instance part="J1" gate="G$1" x="233.68" y="25.4"/>
 <instance part="D1" gate="G$1" x="193.04" y="20.32" rot="R90"/>
-<instance part="SUPPLY4" gate="G$1" x="185.42" y="30.48"/>
 <instance part="GND4" gate="1" x="157.48" y="10.16"/>
 <instance part="LOGO1" gate="G$1" x="15.24" y="68.58"/>
@@
 <instance part="GND8" gate="1" x="40.64" y="208.28"/>
 <instance part="SUPPLY7" gate="G$1" x="246.38" y="71.12" rot="R180"/>
+<instance part="SUPPLY4" gate="G$1" x="185.42" y="30.48"/>
 </instances>
 <busses>
 </busses>
 <nets>
-<net name="VCC" class="0">
-<segment>
-<wire x1="185.42" y1="25.4" x2="185.42" y2="27.94" width="0.1524" layer="91"/>
-<wire x1="185.42" y1="27.94" x2="193.04" y2="27.94" width="0.1524" layer="91"/>
-<pinref part="D1" gate="G$1" pin="C"/>
-<wire x1="193.04" y1="27.94" x2="193.04" y2="22.86" width="0.1524" layer="91"/>
-<wire x1="185.42" y1="27.94" x2="185.42" y2="30.48" width="0.1524" layer="91"/>
-<junction x="185.42" y="27.94"/>
-<pinref part="SUPPLY4" gate="G$1" pin="VCC"/>
-<pinref part="R2" gate="G$1" pin="2"/>
-</segment>
-</net>
 <net name="GND" class="0">
 <segment>
@@
 <pinref part="SUPPLY7" gate="G$1" pin="5V"/>
 </segment>
-</net>
+<segment>
+<wire x1="185.42" y1="25.4" x2="185.42" y2="27.94" width="0.1524" layer="91"/>
+<wire x1="185.42" y1="27.94" x2="193.04" y2="27.94" width="0.1524" layer="91"/>
+<pinref part="D1" gate="G$1" pin="C"/>
+<wire x1="193.04" y1="27.94" x2="193.04" y2="22.86" width="0.1524" layer="91"/>
+<wire x1="185.42" y1="27.94" x2="185.42" y2="30.48" width="0.1524" layer="91"/>
+<junction x="185.42" y="27.94"/>
+<pinref part="R2" gate="G$1" pin="2"/>
+<pinref part="SUPPLY4" gate="G$1" pin="5V"/>
+</segment>
+</net>
