File: PCB/Design1.sch (EAGLE design)
At the start: 40 parts, among them J1 FTDI, U1 ATMEGA2560AU, Y1 16MHZ

Commit message: Labeling Cleanup
Parts:
- renumbered U1 to ATMEGA2560AU, VREG_1 to VREG
Changed lines of the file:
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@@
 </classes>
 <parts>
-<part name="U1" library="SparkFun-DigitalIC" deviceset="ATMEGA2560" device="AU"/>
+<part name="ATMEGA2560AU" library="SparkFun-DigitalIC" deviceset="ATMEGA2560" device="AU" value=""/>
 <part name="GND1" library="SparkFun-Aesthetics" deviceset="GND" device=""/>
 <part name="GND2" library="SparkFun-Aesthetics" deviceset="GND" device=""/>
@@
 <part name="CH_1" library="SparkFun-Connectors" deviceset="M02" device="LOCK_LONGPADS"/>
 <part name="CH_2" library="SparkFun-Connectors" deviceset="M02" device="LOCK_LONGPADS"/>
-<part name="VREG_1" library="SparkFun-PowerIC" deviceset="V_REG_LM1117" device="SOT223"/>
+<part name="VREG" library="SparkFun-PowerIC" deviceset="V_REG_LM1117" device="SOT223"/>
 <part name="C7" library="SparkFun-Capacitors" deviceset="CAP_POL" device="PTH1" value="470uF"/>
 <part name="Y1" library="SparkFun-FreqCtrl" deviceset="RESONATOR" device="16MHZ" value="16MHZ"/>
@@
 </plain>
 <instances>
-<instance part="U1" gate="1" x="144.78" y="139.7"/>
+<instance part="ATMEGA2560AU" gate="1" x="144.78" y="139.7"/>
 <instance part="GND1" gate="1" x="101.6" y="165.1"/>
 <instance part="GND2" gate="1" x="17.78" y="20.32"/>
@@
 <instance part="CH_1" gate="G$1" x="284.48" y="198.12" rot="R180"/>
 <instance part="CH_2" gate="G$1" x="284.48" y="182.88" rot="R180"/>
-<instance part="VREG_1" gate="G$1" x="63.5" y="40.64"/>
+<instance part="VREG" gate="G$1" x="63.5" y="40.64"/>
 <instance part="C7" gate="G$1" x="83.82" y="35.56"/>
 <instance part="Y1" gate="G$1" x="88.9" y="208.28" rot="R270"/>
@@
 <net name="GND" class="0">
 <segment>
-<pinref part="U1" gate="1" pin="GND3"/>
-<pinref part="U1" gate="1" pin="GND2"/>
+<pinref part="ATMEGA2560AU" gate="1" pin="GND3"/>
+<pinref part="ATMEGA2560AU" gate="1" pin="GND2"/>
 <wire x1="109.22" y1="172.72" x2="101.6" y2="172.72" width="0.1524" layer="91"/>
 <junction x="101.6" y="172.72"/>
 <pinref part="GND1" gate="1" pin="GND"/>
-<pinref part="U1" gate="1" pin="GND1"/>
+<pinref part="ATMEGA2560AU" gate="1" pin="GND1"/>
 <wire x1="109.22" y1="175.26" x2="101.6" y2="175.26" width="0.1524" layer="91"/>
-<pinref part="U1" gate="1" pin="GND"/>
-<pinref part="U1" gate="1" pin="AGND"/>
+<pinref part="ATMEGA2560AU" gate="1" pin="GND"/>
+<pinref part="ATMEGA2560AU" gate="1" pin="AGND"/>
 <wire x1="109.22" y1="195.58" x2="101.6" y2="195.58" width="0.1524" layer="91"/>
 <wire x1="101.6" y1="195.58" x2="101.6" y2="177.8" width="0.1524" layer="91"/>
@@
 <junction x="63.5" y="27.94"/>
 <junction x="93.98" y="27.94"/>
-<pinref part="VREG_1" gate="G$1" pin="ADJ"/>
+<pinref part="VREG" gate="G$1" pin="ADJ"/>
 <wire x1="83.82" y1="27.94" x2="93.98" y2="27.94" width="0.1524" layer="91"/>
 <wire x1="63.5" y1="33.02" x2="63.5" y2="27.94" width="0.1524" layer="91"/>
@@
 </segment>
 <segment>
-<pinref part="U1" gate="1" pin="RESET"/>
+<pinref part="ATMEGA2560AU" gate="1" pin="RESET"/>
 <wire x1="109.22" y1="215.9" x2="99.06" y2="215.9" width="0.1524" layer="91"/>
 <label x="99.06" y="215.9" size="1.778" layer="95"/>
@@
 </segment>
 <segment>
-<pinref part="U1" gate="1" pin="(OC0A/OC1C/PCINT7)PB7"/>
+<pinref part="ATMEGA2560AU" gate="1" pin="(OC0A/OC1C/PCINT7)PB7"/>
 <wire x1="180.34" y1="193.04" x2="190.5" y2="193.04" width="0.1524" layer="91"/>
 <label x="182.88" y="193.04" size="1.778" layer="95"/>
@@
 <net name="TX0" class="0">
 <segment>
-<pinref part="U1" gate="1" pin="(TXD0)PE1"/>
+<pinref part="ATMEGA2560AU" gate="1" pin="(TXD0)PE1"/>
 <wire x1="180.34" y1="109.22" x2="187.96" y2="109.22" width="0.1524" layer="91"/>
 <label x="182.88" y="109.22" size="1.778" layer="95"/>
@@
 <net name="RX0" class="0">
 <segment>
-<pinref part="U1" gate="1" pin="(RXD0/PCIN8)PE0"/>
+<pinref part="ATMEGA2560AU" gate="1" pin="(RXD0/PCIN8)PE0"/>
 <wire x1="180.34" y1="106.68" x2="187.96" y2="106.68" width="0.1524" layer="91"/>
 <label x="182.88" y="106.68" size="1.778" layer="95"/>
@@
 <net name="5V" class="0">
 <segment>
-<pinref part="U1" gate="1" pin="VCC"/>
-<pinref part="U1" gate="1" pin="VCC3"/>
-<pinref part="U1" gate="1" pin="VCC2"/>
-<pinref part="U1" gate="1" pin="VCC1"/>
-<pinref part="U1" gate="1" pin="AVCC"/>
+<pinref part="ATMEGA2560AU" gate="1" pin="VCC"/>
+<pinref part="ATMEGA2560AU" gate="1" pin="VCC3"/>
+<pinref part="ATMEGA2560AU" gate="1" pin="VCC2"/>
+<pinref part="ATMEGA2560AU" gate="1" pin="VCC1"/>
+<pinref part="ATMEGA2560AU" gate="1" pin="AVCC"/>
 <wire x1="99.06" y1="198.12" x2="99.06" y2="187.96" width="0.1524" layer="91"/>
 <wire x1="99.06" y1="187.96" x2="99.06" y2="185.42" width="0.1524" layer="91"/>
@@
 <pinref part="C3" gate="G$1" pin="1"/>
 <label x="136.398" y="40.64" size="1.778" layer="95"/>
-<pinref part="VREG_1" gate="G$1" pin="OUT"/>
+<pinref part="VREG" gate="G$1" pin="OUT"/>
 <wire x1="124.46" y1="40.64" x2="144.78" y2="40.64" width="0.1524" layer="91"/>
 <wire x1="71.12" y1="40.64" x2="76.2" y2="40.64" width="0.1524" layer="91"/>
-<pinref part="VREG_1" gate="G$1" pin="OUT@1"/>
+<pinref part="VREG" gate="G$1" pin="OUT@1"/>
 <wire x1="76.2" y1="40.64" x2="83.82" y2="40.64" width="0.1524" layer="91"/>
 <wire x1="83.82" y1="40.64" x2="93.98" y2="40.64" width="0.1524" layer="91"/>
@@
 <net name="TX1" class="0">
 <segment>
-<pinref part="U1" gate="1" pin="(TXD1/INT3)PD3"/>
+<pinref part="ATMEGA2560AU" gate="1" pin="(TXD1/INT3)PD3"/>
 <label x="182.88" y="137.16" size="1.778" layer="95"/>
 <wire x1="187.96" y1="137.16" x2="180.34" y2="137.16" width="0.1524" layer="91"/>
@@
 <net name="RX1" class="0">
 <segment>
-<pinref part="U1" gate="1" pin="(RXD1/INT2)PD2"/>
+<pinref part="ATMEGA2560AU" gate="1" pin="(RXD1/INT2)PD2"/>
 <label x="182.88" y="134.62" size="1.778" layer="95"/>
 <wire x1="187.96" y1="134.62" x2="180.34" y2="134.62" width="0.1524" layer="91"/>
@@
 <net name="TX2" class="0">
 <segment>
-<pinref part="U1" gate="1" pin="PH1(TXD2)"/>
+<pinref part="ATMEGA2560AU" gate="1" pin="PH1(TXD2)"/>
 <wire x1="104.14" y1="68.58" x2="109.22" y2="68.58" width="0.1524" layer="91"/>
 <label x="104.14" y="68.58" size="1.778" layer="95"/>
@@
 <net name="RX2" class="0">
 <segment>
-<pinref part="U1" gate="1" pin="PH0(RXD2)"/>
+<pinref part="ATMEGA2560AU" gate="1" pin="PH0(RXD2)"/>
 <wire x1="104.14" y1="66.04" x2="109.22" y2="66.04" width="0.1524" layer="91"/>
 <label x="104.14" y="66.04" size="1.778" layer="95"/>
@@
 </segment>
 <segment>
-<pinref part="U1" gate="1" pin="(ADC0)PF0"/>
+<pinref part="ATMEGA2560AU" gate="1" pin="(ADC0)PF0"/>
 <wire x1="180.34" y1="83.82" x2="193.04" y2="83.82" width="0.1524" layer="91"/>
 <label x="182.88" y="83.82" size="1.778" layer="95"/>
@@
 </segment>
 <segment>
-<pinref part="U1" gate="1" pin="(SCK/PCINT1)PB1"/>
+<pinref part="ATMEGA2560AU" gate="1" pin="(SCK/PCINT1)PB1"/>
 <wire x1="180.34" y1="177.8" x2="190.5" y2="177.8" width="0.1524" layer="91"/>
 <label x="182.88" y="177.8" size="1.778" layer="95"/>
@@
 </segment>
 <segment>
-<pinref part="U1" gate="1" pin="(MISO/PCINT3)PB3"/>
+<pinref part="ATMEGA2560AU" gate="1" pin="(MISO/PCINT3)PB3"/>
 <wire x1="180.34" y1="182.88" x2="190.5" y2="182.88" width="0.1524" layer="91"/>
 <label x="182.88" y="182.88" size="1.778" layer="95"/>
@@
 </segment>
 <segment>
-<pinref part="U1" gate="1" pin="(MOSI/PCINT2)PB2"/>
+<pinref part="ATMEGA2560AU" gate="1" pin="(MOSI/PCINT2)PB2"/>
 <wire x1="180.34" y1="180.34" x2="190.5" y2="180.34" width="0.1524" layer="91"/>
 <label x="182.88" y="180.34" size="1.778" layer="95"/>
@@
 </segment>
 <segment>
-<pinref part="U1" gate="1" pin="PH7(T4)"/>
+<pinref part="ATMEGA2560AU" gate="1" pin="PH7(T4)"/>
 <wire x1="109.22" y1="83.82" x2="96.52" y2="83.82" width="0.1524" layer="91"/>
 <label x="96.52" y="83.82" size="1.778" layer="95"/>
@@
 </segment>
 <segment>
-<pinref part="U1" gate="1" pin="(TOSC2)PG3"/>
+<pinref part="ATMEGA2560AU" gate="1" pin="(TOSC2)PG3"/>
 <wire x1="180.34" y1="73.66" x2="193.04" y2="73.66" width="0.1524" layer="91"/>
 <label x="182.88" y="73.66" size="1.778" layer="95"/>
@@
 <wire x1="35.56" y1="38.1" x2="35.56" y2="40.64" width="0.1524" layer="91"/>
 <junction x="35.56" y="40.64"/>
-<pinref part="VREG_1" gate="G$1" pin="IN"/>
+<pinref part="VREG" gate="G$1" pin="IN"/>
 </segment>
 </net>
@@
 <segment>
 <pinref part="Y1" gate="G$1" pin="1"/>
-<pinref part="U1" gate="1" pin="XTAL2"/>
+<pinref part="ATMEGA2560AU" gate="1" pin="XTAL2"/>
 <wire x1="109.22" y1="210.82" x2="88.9" y2="210.82" width="0.1524" layer="91"/>
 <wire x1="88.9" y1="210.82" x2="88.9" y2="215.9" width="0.1524" layer="91"/>
@@
 <segment>
 <pinref part="Y1" gate="G$1" pin="3"/>
-<pinref part="U1" gate="1" pin="XTAL1"/>
+<pinref part="ATMEGA2560AU" gate="1" pin="XTAL1"/>
 <wire x1="109.22" y1="205.74" x2="88.9" y2="205.74" width="0.1524" layer="91"/>
 <wire x1="88.9" y1="205.74" x2="88.9" y2="200.66" width="0.1524" layer="91"/>
@@
 <net name="SDA" class="0">
 <segment>
-<pinref part="U1" gate="1" pin="(SDA/INT1)PD1"/>
+<pinref part="ATMEGA2560AU" gate="1" pin="(SDA/INT1)PD1"/>
 <wire x1="180.34" y1="132.08" x2="190.5" y2="132.08" width="0.1524" layer="91"/>
 <label x="182.88" y="132.08" size="1.778" layer="95"/>
@@
 <net name="SCL" class="0">
 <segment>
-<pinref part="U1" gate="1" pin="(SCL/INT0)PD0"/>
+<pinref part="ATMEGA2560AU" gate="1" pin="(SCL/INT0)PD0"/>
 <wire x1="190.5" y1="129.54" x2="180.34" y2="129.54" width="0.1524" layer="91"/>
 <label x="182.88" y="129.54" size="1.778" layer="95"/>
@@
 <net name="ADC14" class="0">
 <segment>
-<pinref part="U1" gate="1" pin="PK6(ADC14/PCINT22)"/>
+<pinref part="ATMEGA2560AU" gate="1" pin="PK6(ADC14/PCINT22)"/>
 <wire x1="109.22" y1="127" x2="99.06" y2="127" width="0.1524" layer="91"/>
 <label x="99.06" y="127" size="1.778" layer="95"/>
@@
 <net name="ADC15" class="0">
 <segment>
-<pinref part="U1" gate="1" pin="PK7(ADC15/PCINT23)"/>
+<pinref part="ATMEGA2560AU" gate="1" pin="PK7(ADC15/PCINT23)"/>
 <wire x1="109.22" y1="129.54" x2="99.06" y2="129.54" width="0.1524" layer="91"/>
 <label x="99.06" y="129.54" size="1.778" layer="95"/>
