File: PCB/RocketDuino.brd (EAGLE design)
At the start: 73 x 41 mm, 42 parts, among them J1 FTDI, Y1 16MHZ

Commit message: Revert "Add Labels (2)"
This reverts commit 649e5ca491e825c42b75eb8464ca0d71b423613b.
Parts:
- renumbered INFO to 13
Other:
- board text removed: "GND RX TX 5V"
- board text removed: "GND TX RX 5V"
- board text removed: "Serial 1"
- board text removed: "Serial 2"
Changed lines of the file:
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@@
 <wire x1="69" y1="2" x2="71" y2="0" width="0.127" layer="20" curve="-90"/>
 <wire x1="67" y1="0" x2="69" y2="2" width="0.127" layer="20" curve="-90"/>
-<text x="30" y="3" size="0.8128" layer="21">GND  RX   TX    5V</text>
-<text x="3" y="12.5" size="0.8128" layer="21">GND  TX   RX    5V</text>
-<text x="28.5" y="9" size="1.016" layer="21" rot="R270">Serial 1</text>
-<text x="1.5" y="11.25" size="1.016" layer="21" rot="R270">Serial 2</text>
 </plain>
 <attributes>
@@
 <element name="D1" library="SparkFun-DiscreteSemi" package="SMA-DIODE_ALT" value="" x="12" y="32" rot="R180"/>
 <element name="LOGO1" library="SparkFun-Aesthetics" package="OSHW-LOGO-M" value="OSHW-LOGOM" x="18.5" y="36.98"/>
-<element name="INFO" library="led" package="SML0805" value="" x="20.5" y="6" rot="R90"/>
+<element name="13" library="led" package="SML0805" value="" x="20.5" y="6" rot="R90"/>
 <element name="MOS" library="SparkFun-Connectors" package="1X02_LOCK_LONGPADS" value="" x="70.75" y="18.25" locked="yes" smashed="yes" rot="R180">
 <attribute name="NAME" x="65.778" y="19.27" size="0.8128" layer="25" font="vector" rot="R270"/>
@@
 <contactref element="J1" pad="P$6"/>
 <contactref element="J1" pad="P$5"/>
-<contactref element="INFO" pad="C"/>
+<contactref element="13" pad="C"/>
 <contactref element="ATMEGA2560AU" pad="32"/>
 <contactref element="ATMEGA2560AU" pad="11"/>
@@
 </signal>
 <signal name="N$3">
-<contactref element="INFO" pad="A"/>
+<contactref element="13" pad="A"/>
 <contactref element="R4" pad="1"/>
 <wire x1="20.5" y1="9.6" x2="20.5" y2="7.05" width="0.3" layer="1"/>
